File: ElectronicDesigns/Test_antenna/RFID_Eval_13.56MHz-v14.brd (EAGLE design)
At the start: 2.5 x 53.3 mm, 22 parts, among them U1 TLV1117-18IDCYG3

Commit message: Circuit modified for antenna of Sparkfun
Parts:
- removed JP10, JP13, JP3, JP5, JP7: STAND-OFF, SparkFun:STAND-OFF
- removed JP12: FIDUCIAL1X2, SparkFun:FIDUCIAL-1X2
- removed JP8: LOGO-SFENEW, SparkFun:SFE-NEW-WEBLOGO
- moved U$1 18.0 mm to (29.0, 25.9)
- moved C2 18.0 mm to (39.3, 28.4)
- moved C3 18.0 mm to (41.7, 25.9)
- moved C4 18.0 mm to (41.7, 28.4)
- moved C5 18.0 mm to (39.3, 25.9)
- moved C6 18.0 mm to (39.3, 29.7)
- moved C7 18.0 mm to (39.3, 24.6)
- moved C8 18.0 mm to (18.1, 25.6)
- moved R1 18.0 mm to (6.70, 28.2)
- moved R8 18.0 mm to (41.7, 24.6)
- moved R9 18.0 mm to (41.7, 29.7)
- moved U$2 18.0 mm to (20.1, 31.0)
- moved U$3 18.0 mm to (11.8, 28.3)
- moved U1 18.0 mm to (-3.09, 28.3)
- moved C1 18.0 mm to (31.0, 30.2)
Routing:
- net GND: track 559.6 -> 522.6 mm
- net N$8: track 534.8 -> 532.7 mm
Other:
- board outline removed
- board text removed: "13.56 MHz"
- board text removed: "A5"
- board text removed: "RFID Eval"
- board text removed: "RX"
