File: ElectronicDesigns/Test_antenna/RFID_Eval_13.56MHz-v14.sch (EAGLE design)
At the start: 22 parts, among them U1 TLV1117-18IDCYG3

Commit message: Circuit modified for antenna of Sparkfun
Parts:
- removed JP10, JP13, JP3, JP5, JP7: STAND-OFF, SparkFun:STAND-OFF
- removed JP12: FIDUCIAL1X2, SparkFun:FIDUCIAL1X2
- removed JP8: LOGO-SFENEW, SparkFun:LOGO-SFENEW
Changed lines of the file:
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@@
 <parts>
 <part name="FRAME1" library="SparkFun" deviceset="FRAME-LETTER" device=""/>
-<part name="JP3" library="SparkFun" deviceset="STAND-OFF" device=""/>
 <part name="R8" library="SparkFun" deviceset="RESISTOR" device="0402-RES" value="0 Ohm"/>
 <part name="R9" library="SparkFun" deviceset="RESISTOR" device="0402-RES" value="0 Ohm"/>
@@
 <part name="C6" library="SparkFun" deviceset="CAP" device="0402-CAP" value="18pF"/>
 <part name="GND10" library="SparkFun" deviceset="GND" device=""/>
-<part name="JP5" library="SparkFun" deviceset="STAND-OFF" device=""/>
-<part name="JP7" library="SparkFun" deviceset="STAND-OFF" device=""/>
-<part name="JP8" library="SparkFun" deviceset="LOGO-SFE" device="NEW"/>
-<part name="JP12" library="SparkFun" deviceset="FIDUCIAL" device="1X2"/>
-<part name="JP10" library="SparkFun" deviceset="STAND-OFF" device=""/>
-<part name="JP13" library="SparkFun" deviceset="STAND-OFF" device=""/>
 <part name="C2" library="SparkFun" deviceset="CAP" device="0402-CAP" value="22pF"/>
 <part name="C7" library="SparkFun" deviceset="CAP" device="0402-CAP" value="22pF"/>
@@
 <instance part="FRAME1" gate="G$1" x="0" y="0"/>
 <instance part="FRAME1" gate="G$2" x="147.32" y="0"/>
-<instance part="JP3" gate="G$1" x="236.22" y="33.02"/>
 <instance part="R8" gate="G$1" x="111.76" y="66.04" rot="R180"/>
 <instance part="R9" gate="G$1" x="111.76" y="60.96" rot="R180"/>
@@
 <instance part="C6" gate="G$1" x="76.2" y="60.96" rot="R90"/>
 <instance part="GND10" gate="1" x="104.14" y="43.18"/>
-<instance part="JP5" gate="G$1" x="241.3" y="33.02"/>
-<instance part="JP7" gate="G$1" x="246.38" y="33.02"/>
-<instance part="JP8" gate="G$1" x="241.3" y="25.4"/>
-<instance part="JP12" gate="G$1" x="215.9" y="25.4"/>
-<instance part="JP10" gate="G$1" x="226.06" y="33.02"/>
-<instance part="JP13" gate="G$1" x="231.14" y="33.02"/>
 <instance part="C2" gate="G$1" x="81.28" y="53.34" smashed="yes">
 <attribute name="NAME" x="77.724" y="56.261" size="1.778" layer="95"/>
