File: Designs/ElectronicDesigns/Final_v2_NCP161_ 711AJ/Final_v2.brd (EAGLE design)
At the start: 47.1 x 23.1 mm, 5 parts

Commit message: gui guidebook
Parts:
- moved R1 5.41 mm to (22.9, 11.3)
- moved C1 1.53 mm to (14.7, 10.4)
- moved U$2 1.53 mm to (14.1, 8.00)
- moved U$3 1.53 mm to (19.2, 10.3)
- moved D1 1.53 mm to (43.2, 13.0)
Routing:
- net OUT: track 7.71 -> 2.81 mm
- net N$2: track 14.6 -> 19.5 mm

Commit message: changes
Routing:
- net N$403: track 0.00 -> 752.8 mm
- net N$305: track 0.00 -> 547.0 mm
- net N$271: track 0.00 -> 448.9 mm
- net N$222: track 0.00 -> 363.5 mm
- net N$233: track 0.00 -> 353.0 mm
- net N$437: track 0.00 -> 341.4 mm
- net N$353: track 0.00 -> 279.6 mm
- net N$363: track 0.00 -> 267.5 mm
- net N$343: track 0.00 -> 246.6 mm
- net N$312: track 0.00 -> 241.2 mm
- net N$331: track 0.00 -> 239.1 mm
- net N$371: track 0.00 -> 226.2 mm
- net N$320: track 0.00 -> 197.7 mm
- net N$960: track 0.00 -> 187.3 mm
- net N$297: track 0.00 -> 179.6 mm
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