File: Designs/Electronic_Design/Final_v2_NCP161_antenna/Final_v2.brd (EAGLE design)
At the start: 100 x 31.8 mm, 5 parts

Commit message: Printings
Routing:
- net N$1: track 3.37 -> 0.00 mm
Other:
- board text removed: "Matching capacitor"
Changed lines of the file:
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@@
 <wire x1="100" y1="31.81" x2="0" y2="31.81" width="0" layer="20"/>
 <wire x1="0" y1="31.81" x2="0" y2="0" width="0" layer="20"/>
-<wire x1="90.6" y1="10" x2="50.6" y2="10" width="0.1524" layer="21"/>
-<dimension x1="90.6" y1="10" x2="50.6" y2="10" x3="70.6" y3="1.3" textsize="1.778" layer="21"/>
-<text x="32.7" y="23.7" size="1.778" layer="1">Matching capacitor</text>
+<wire x1="4" y1="6" x2="4" y2="27.4" width="0.1524" layer="21"/>
+<dimension x1="4" y1="6" x2="4" y2="27.4" x3="-3.5" y3="16.7" textsize="1.778" layer="21"/>
+<wire x1="6.7" y1="4.9" x2="93.1" y2="4.9" width="0.1524" layer="21"/>
+<dimension x1="6.7" y1="4.9" x2="28.9" y2="4.9" x3="17.8" y3="1.6" textsize="1.778" layer="21"/>
+<dimension x1="6.7" y1="4.9" x2="50.6" y2="4.9" x3="28.65" y3="-4.4" textsize="1.778" layer="21"/>
+<wire x1="93.1" y1="4.9" x2="93.1" y2="5" width="0.1524" layer="21"/>
+<dimension x1="93.1" y1="4.9" x2="6.7" y2="4.9" x3="49.9" y3="-12.4" textsize="1.778" layer="21"/>
+<wire x1="96.1" y1="13.1" x2="96.1" y2="20" width="0.1524" layer="21"/>
+<dimension x1="96.1" y1="13.1" x2="96.1" y2="20" x3="108.4" y3="16.55" textsize="1.778" layer="21"/>
 </plain>
 <attributes>
@@
 <wire x1="35.3" y1="15" x2="35.3" y2="15.6" width="0.5" layer="1"/>
 </signal>
-<signal name="N$1">
-<wire x1="35.6" y1="21.8" x2="35.6" y2="19.9" width="0.5" layer="1"/>
-<wire x1="35.1" y1="20.4" x2="35.6" y2="19.9" width="0.5" layer="1"/>
-<wire x1="35.6" y1="19.9" x2="35.7" y2="19.9" width="0.5" layer="1"/>
-<wire x1="35.7" y1="19.9" x2="36.1" y2="20.3" width="0.5" layer="1"/>
-<wire x1="36.1" y1="20.3" x2="36.1" y2="20.4" width="0.5" layer="1"/>
-</signal>
 </signals>
