File: Designs/Electronic_Design/Final_NCP161_Package1_antenna_8MHz/Final_v2.brd (EAGLE design)
At the start: 100 x 68.1 mm, 5 parts

Commit message: Printing
Routing:
- net GND1: track 464.1 -> 0.00 mm
- net IN+: track 542.7 -> 276.1 mm, vias 0 -> 2
